Commit message: update urdf with dae files and gazebo update

File: turtlebot3_description/urdf/turtlebot3_big_wheel.urdf.xacro (robot description, xacro)
@@ -6,5 +6,5 @@
   <xacro:arg name="publish_pointcloud" default="false" />
   <xacro:include filename="$(find turtlebot3_description)/urdf/common_properties.urdf"/>
-  <!-- <xacro:include filename="$(find turtlebot3_description)/urdf/turtlebot3_big_wheel.gazebo.xacro"/> -->
+  <xacro:include filename="$(find turtlebot3_description)/urdf/turtlebot3_big_wheel.gazebo.xacro"/>
   <xacro:include filename="$(find realsense2_description)/urdf/_d435.urdf.xacro" />
   <link name="base_footprint"/>
@@ -18,5 +18,5 @@
       <origin xyz="-0.064 0 0" rpy="0 0 0"/>
       <geometry>
-        <mesh filename="package://turtlebot3_description/meshes/bases/waffle_pi_base.stl" scale="0.001 0.001 0.001"/>
+        <mesh filename="package://turtlebot3_description/meshes/bases/waffle_pi_base.dae" scale="0.001 0.001 0.001"/>
       </geometry>
       <material name="light_black"/>
@@ -101,5 +101,5 @@
       <origin xyz="0 0.00175 0" rpy="1.57 0 0"/>
       <geometry>
-        <mesh filename="package://turtlebot3_description/meshes/joints/big_wheel_caster_joint.stl" scale="0.001 0.001 0.001"/>
+        <mesh filename="package://turtlebot3_description/meshes/joints/big_wheel_caster_joint.dae" scale="0.001 0.001 0.001"/>
       </geometry>
       <material name="dark"/>
@@ -128,5 +128,5 @@
       <origin xyz="0 0.00175 0" rpy="1.57 0 0"/>
       <geometry>
-        <mesh filename="package://turtlebot3_description/meshes/joints/big_wheel_caster_joint.stl" scale="0.001 0.001 0.001"/>
+        <mesh filename="package://turtlebot3_description/meshes/joints/big_wheel_caster_joint.dae" scale="0.001 0.001 0.001"/>
       </geometry>
       <material name="dark"/>
@@ -161,5 +161,5 @@
       <origin xyz="0 0 0.0" rpy="0 0 0"/>
       <geometry>
-        <mesh filename="package://turtlebot3_description/meshes/sensors/lds.stl" scale="0.001 0.001 0.001"/>
+        <mesh filename="package://turtlebot3_description/meshes/sensors/lds.dae" scale="0.001 0.001 0.001"/>
       </geometry>
       <material name="dark"/>
@@ -188,5 +188,5 @@
       <origin xyz="0 0 0.0" rpy="0 0 1.57"/>
       <geometry>
-        <mesh filename="package://turtlebot3_description/meshes/joints/d435_base_camera.stl" scale="0.001 0.001 0.001"/>
+        <mesh filename="package://turtlebot3_description/meshes/joints/d435_base_camera.dae" scale="0.001 0.001 0.001"/>
       </geometry>
       <material name="light_black"/>

Commit message: update path to ros2 format

File: turtlebot3_description/urdf/turtlebot3_big_wheel.urdf.xacro (robot description, xacro)
@@ -1,4 +1,4 @@
 <?xml version="1.0" ?>
-<robot name="turtlebot3_big_wheel" xmlns:xacro="http://ros.org/wiki/xacro">
+<robot name="turtlebot3_big_wheel" xmlns:xacro="http://www.ros.org/wiki/xacro">
   <xacro:arg name="use_nominal_extrinsics" default="true"/>
   <xacro:arg name="add_plug" default="false" />
@@ -18,5 +18,6 @@
       <origin xyz="-0.064 0 0" rpy="0 0 0"/>
       <geometry>
-        <mesh filename="package://turtlebot3_description/meshes/bases/waffle_pi_base.dae" scale="0.001 0.001 0.001"/>
+        <mesh filename="$(find turtlebot3_description)/meshes/bases/waffle_pi_base.dae" scale="0.001 0.001 0.001"/>
+        <!-- <mesh filename="$(find turtlebot3_description)/meshes/bases/big_wheel_base.dae" scale="0.001 0.001 0.001"/> -->
       </geometry>
       <material name="light_black"/>
@@ -46,5 +47,5 @@
       <origin xyz="0 0 0" rpy="0 0 0"/>
       <geometry>
-        <mesh filename="package://turtlebot3_description/meshes/wheels/big_wheel_tire.dae" scale="1.00 1.00 1.00"/>
+        <mesh filename="$(find turtlebot3_description)/meshes/wheels/big_wheel_tire.dae" scale="1.00 1.00 1.00"/>
       </geometry>
       <material name="dark"/>
@@ -74,5 +75,5 @@
       <origin xyz="0 0 0" rpy="0 0 0"/>
       <geometry>
-        <mesh filename="package://turtlebot3_description/meshes/wheels/big_wheel_tire.dae" scale="1.00 1.00 1.00"/>
+        <mesh filename="$(find turtlebot3_description)/meshes/wheels/big_wheel_tire.dae" scale="1.00 1.00 1.00"/>
       </geometry>
       <material name="dark"/>
@@ -101,5 +102,5 @@
       <origin xyz="0 0.00175 0" rpy="1.57 0 0"/>
       <geometry>
-        <mesh filename="package://turtlebot3_description/meshes/joints/big_wheel_caster_joint.dae" scale="0.001 0.001 0.001"/>
+        <mesh filename="$(find turtlebot3_description)/meshes/joints/big_wheel_caster_joint.dae" scale="0.001 0.001 0.001"/>
       </geometry>
       <material name="dark"/>
@@ -128,5 +129,5 @@
       <origin xyz="0 0.00175 0" rpy="1.57 0 0"/>
       <geometry>
-        <mesh filename="package://turtlebot3_description/meshes/joints/big_wheel_caster_joint.dae" scale="0.001 0.001 0.001"/>
+        <mesh filename="$(find turtlebot3_description)/meshes/joints/big_wheel_caster_joint.dae" scale="0.001 0.001 0.001"/>
       </geometry>
       <material name="dark"/>
@@ -161,5 +162,5 @@
       <origin xyz="0 0 0.0" rpy="0 0 0"/>
       <geometry>
-        <mesh filename="package://turtlebot3_description/meshes/sensors/lds.dae" scale="0.001 0.001 0.001"/>
+        <mesh filename="$(find turtlebot3_description)/meshes/sensors/lds.stl" scale="0.001 0.001 0.001"/>
       </geometry>
       <material name="dark"/>
@@ -188,5 +189,5 @@
       <origin xyz="0 0 0.0" rpy="0 0 1.57"/>
       <geometry>
-        <mesh filename="package://turtlebot3_description/meshes/joints/d435_base_camera.dae" scale="0.001 0.001 0.001"/>
+        <mesh filename="$(find turtlebot3_description)/meshes/joints/d435_base_camera.dae" scale="0.001 0.001 0.001"/>
       </geometry>
       <material name="light_black"/>
