Commit message: update urdf files for xacro support in humble

File: turtlebot3_description/urdf/common_properties.urdf.xacro (robot description, xacro)
@@ -1,5 +1,4 @@
 <?xml version="1.0" ?>
-<robot name="xacro_properties"
-  xmlns:xacro="http://ros.org/wiki/xacro">
+<robot name="xacro_properties" xmlns:xacro="http://ros.org/wiki/xacro">
   <!-- Init colour -->
   <material name="black">
@@ -22,8 +21,8 @@
   </material>
   <material name="orange">
-    <color rgba="1.0 0.423529412 0.039215686 1.0"/>
+    <color rgba="${255/255} ${108/255} ${10/255} 1.0"/>
   </material>
   <material name="brown">
-    <color rgba="0.870588235 0.811764706 0.764705882 1.0"/>
+    <color rgba="${222/255} ${207/255} ${195/255} 1.0"/>
   </material>
   <material name="red">

File: turtlebot3_description/urdf/turtlebot3_big_wheel.gazebo.xacro (robot description, xacro)
@@ -126,4 +126,15 @@
       <odometry_frame>odom</odometry_frame>
       <robot_base_frame>base_footprint</robot_base_frame>
+    </plugin>
+  </gazebo>
+  <gazebo>
+    <plugin name="turtlebot3_joint_state" filename="libgazebo_ros_joint_state_publisher.so">
+      <ros>
+        <!-- <namespace>/tb3</namespace> -->
+        <remapping>~/out:=joint_states</remapping>
+      </ros>
+      <update_rate>30</update_rate>
+      <joint_name>wheel_left_joint</joint_name>
+      <joint_name>wheel_right_joint</joint_name>
     </plugin>
   </gazebo>

File: turtlebot3_description/urdf/turtlebot3_big_wheel.urdf.xacro (robot description, xacro)
@@ -5,5 +5,5 @@
   <xacro:arg name="use_mesh" default="true" />
   <xacro:arg name="publish_pointcloud" default="false" />
-  <xacro:include filename="$(find turtlebot3_description)/urdf/common_properties.urdf"/>
+  <xacro:include filename="$(find turtlebot3_description)/urdf/common_properties.urdf.xacro"/>
   <xacro:include filename="$(find turtlebot3_description)/urdf/turtlebot3_big_wheel.gazebo.xacro"/>
   <xacro:include filename="$(find realsense2_description)/urdf/_d435.urdf.xacro" />
@@ -18,6 +18,6 @@
       <origin xyz="-0.064 0 0" rpy="0 0 0"/>
       <geometry>
-        <mesh filename="$(find turtlebot3_description)/meshes/bases/waffle_pi_base.dae" scale="0.001 0.001 0.001"/>
-        <!-- <mesh filename="$(find turtlebot3_description)/meshes/bases/big_wheel_base.dae" scale="0.001 0.001 0.001"/> -->
+        <mesh filename="file://$(find turtlebot3_description)/meshes/bases/waffle_pi_base.dae" scale="0.001 0.001 0.001"/>
+        <!-- <mesh filename="file://$(find turtlebot3_description)/meshes/bases/big_wheel_base.dae" scale="0.001 0.001 0.001"/> -->
       </geometry>
       <material name="light_black"/>
@@ -47,7 +47,7 @@
       <origin xyz="0 0 0" rpy="0 0 0"/>
       <geometry>
-        <mesh filename="$(find turtlebot3_description)/meshes/wheels/big_wheel_tire.dae" scale="1.00 1.00 1.00"/>
-      </geometry>
-      <material name="dark"/>
+        <mesh filename="file://$(find turtlebot3_description)/meshes/wheels/big_wheel_tire.dae" scale="1.00 1.00 1.00"/>
+      </geometry>
+      <material name="orange"/>
     </visual>
     <collision>
@@ -75,7 +75,7 @@
       <origin xyz="0 0 0" rpy="0 0 0"/>
       <geometry>
-        <mesh filename="$(find turtlebot3_description)/meshes/wheels/big_wheel_tire.dae" scale="1.00 1.00 1.00"/>
-      </geometry>
-      <material name="dark"/>
+        <mesh filename="file://$(find turtlebot3_description)/meshes/wheels/big_wheel_tire.dae" scale="1.00 1.00 1.00"/>
+      </geometry>
+      <material name="orange"/>
     </visual>
     <collision>
@@ -102,10 +102,10 @@
       <origin xyz="0 0.00175 0" rpy="1.57 0 0"/>
       <geometry>
-        <mesh filename="$(find turtlebot3_description)/meshes/joints/big_wheel_caster_joint.dae" scale="0.001 0.001 0.001"/>
+        <mesh filename="file://$(find turtlebot3_description)/meshes/joints/big_wheel_caster_joint.dae" scale="0.001 0.001 0.001"/>
       </geometry>
       <material name="dark"/>
     </visual>
     <collision>
-      <origin xyz="0 ${0.039/2} 0" rpy="1.57 0 0"/>
+      <origin xyz="0 0.0185 0" rpy="1.57 0 0"/>
       <geometry>
         <box size="0.030 0.009 0.039"/>
@@ -129,10 +129,10 @@
       <origin xyz="0 0.00175 0" rpy="1.57 0 0"/>
       <geometry>
-        <mesh filename="$(find turtlebot3_description)/meshes/joints/big_wheel_caster_joint.dae" scale="0.001 0.001 0.001"/>
+        <mesh filename="file://$(find turtlebot3_description)/meshes/joints/big_wheel_caster_joint.dae" scale="0.001 0.001 0.001"/>
       </geometry>
       <material name="dark"/>
     </visual>
     <collision>
-      <origin xyz="0 ${0.039/2} 0" rpy="1.57 0 0"/>
+      <origin xyz="0 0.0185 0" rpy="1.57 0 0"/>
       <geometry>
         <box size="0.030 0.009 0.039"/>
@@ -162,5 +162,5 @@
       <origin xyz="0 0 0.0" rpy="0 0 0"/>
       <geometry>
-        <mesh filename="$(find turtlebot3_description)/meshes/sensors/lds.stl" scale="0.001 0.001 0.001"/>
+        <mesh filename="file://$(find turtlebot3_description)/meshes/sensors/lds.stl" scale="0.001 0.001 0.001"/>
       </geometry>
       <material name="dark"/>
@@ -189,5 +189,5 @@
       <origin xyz="0 0 0.0" rpy="0 0 1.57"/>
       <geometry>
-        <mesh filename="$(find turtlebot3_description)/meshes/joints/d435_base_camera.dae" scale="0.001 0.001 0.001"/>
+        <mesh filename="file://$(find turtlebot3_description)/meshes/joints/d435_base_camera.dae" scale="0.001 0.001 0.001"/>
       </geometry>
       <material name="light_black"/>
