Commit message: update tb3_puntilt.urdf moving puntilt to center

File: turtlebot3_description/urdf/turtlebot3_burger_puntilt.urdf.xacro (robot description, xacro)
@@ -1,4 +1,4 @@
 <?xml version="1.0" ?>
-<robot name="turtlebot3_burger" xmlns:xacro="http://ros.org/wiki/xacro">
+<robot name="turtlebot3_burger_puntilt" xmlns:xacro="http://ros.org/wiki/xacro">
   <xacro:include filename="$(find turtlebot3_description)/urdf/common_properties.xacro"/>
   <xacro:include filename="$(find turtlebot3_description)/urdf/turtlebot3_burger_puntilt.gazebo.xacro"/>
@@ -32,7 +32,7 @@
       <origin xyz="0 0 0" rpy="0 0 0"/>
       <mass value="8.2573504e-01"/>
-      <inertia ixx="2.2124416e-03" ixy="-1.2294101e-05" ixz="3.4938785e-05"
-               iyy="2.1193702e-03" iyz="-5.0120904e-06"
-               izz="2.0064271e-03" />
+      <inertia ixx="2.2124416e-03" ixy="-1.2294101e-05" ixz=" 3.4938785e-05"
+                                   iyy=" 2.1193702e-03" iyz="-5.0120904e-06"
+                                                        izz=" 2.0064271e-03" />
     </inertial>
   </link>
@@ -61,6 +61,6 @@
       <mass value="2.8498940e-02" />
       <inertia ixx="1.1175580e-05" ixy="-4.2369783e-11" ixz="-5.9381719e-09"
-               iyy="1.1192413e-05" iyz="-1.4400107e-11"
-               izz="2.0712558e-05" />
+                                   iyy=" 1.1192413e-05" iyz="-1.4400107e-11"
+                                                        izz=" 2.0712558e-05" />
       </inertial>
   </link>
@@ -89,6 +89,6 @@
       <mass value="2.8498940e-02" />
       <inertia ixx="1.1175580e-05" ixy="-4.2369783e-11" ixz="-5.9381719e-09"
-               iyy="1.1192413e-05" iyz="-1.4400107e-11"
-               izz="2.0712558e-05" />
+                                   iyy=" 1.1192413e-05" iyz="-1.4400107e-11"
+                                                        izz=" 2.0712558e-05" />
       </inertial>
   </link>
@@ -142,14 +142,14 @@
       <mass value="0.114" />
       <origin xyz="0 0 0" />
-      <inertia ixx="0.001" ixy="0.0" ixz="0.0"
-               iyy="0.001" iyz="0.0"
-               izz="0.001" />
+      <inertia ixx="0.001" ixy="0.0"   ixz="0.0"
+                           iyy="0.001" iyz="0.0"
+                                       izz="0.001" />
     </inertial>
   </link>
-  <!--* Sensor -->
+  <!--* Realsense -->
   <joint name="puntilt_base" type="fixed">
 		<parent link="base_link"/>
 		<child link="base_puntilt"/>
-		<origin xyz="0.015 0.0 0.171" rpy="0 0 ${-pi/2}"/>
+		<origin xyz="-0.032 0.0 ${0.171 + 0.02}" rpy="0 0 ${-pi/2}"/>
 	</joint>
 	<link name="base_puntilt"/>
