Commit message: update burger_pantilt

File: turtlebot3_description/urdf/turtlebot3_burger_puntilt.gazebo.xacro (robot description, xacro)
@@ -124,3 +124,9 @@
     </sensor>
   </gazebo>
+  <!-- <gazebo>
+    <plugin name="control" filename="libgazebo_ros_control.so"/>
+    <plugin name="joint_state_publisher" filename="libgazebo_ros_joint_state_publisher.so">
+      <jointName>base_puntilt_joint, base_realsense_joint</jointName>
+    </plugin>
+  </gazebo> -->
 </robot>

File: turtlebot3_description/urdf/turtlebot3_burger_puntilt.urdf.xacro (robot description, xacro)
@@ -2,5 +2,11 @@
 <robot name="turtlebot3_burger" xmlns:xacro="http://ros.org/wiki/xacro">
   <xacro:include filename="$(find turtlebot3_description)/urdf/common_properties.xacro"/>
-  <xacro:include filename="$(find turtlebot3_description)/urdf/turtlebot3_burger.gazebo.xacro"/>
+  <xacro:include filename="$(find turtlebot3_description)/urdf/turtlebot3_burger_puntilt.gazebo.xacro"/>
+  <xacro:include filename="$(find realsense2_description)/urdf/_d435.urdf.xacro" />
+	<xacro:include filename="$(find turtlebot3_description)/urdf/_2XL430.urdf.xacro"/>
+  <!-- realsense 関連の引数 -->
+  <xacro:arg name="use_nominal_extrinsics" default="true"/>
+  <xacro:arg name="add_plug" default="false" />
+  <xacro:arg name="use_mesh" default="true" />
   <link name="base_footprint"/>
   <joint name="base_joint" type="fixed">
@@ -107,4 +113,5 @@
     </inertial>
   </link>
+  <!--* Sensor -->
   <joint name="imu_joint" type="fixed">
     <parent link="base_link"/>
@@ -140,3 +147,15 @@
     </inertial>
   </link>
+  <!--* Sensor -->
+  <joint name="puntilt_base" type="fixed">
+		<parent link="base_link"/>
+		<child link="base_puntilt"/>
+		<origin xyz="0.015 0.0 0.171" rpy="0 0 ${-pi/2}"/>
+	</joint>
+	<link name="base_puntilt"/>
+	<xacro:motor_2XL430 parent="base_puntilt" center_parent="false" child="base_realsense" center_child="true" />
+	<link name="base_realsense"/>
+  <xacro:sensor_d435 parent="base_realsense" use_nominal_extrinsics="$(arg use_nominal_extrinsics)" add_plug="$(arg add_plug)" use_mesh="$(arg use_mesh)">
+    <origin xyz="-0.01 -0.035 0.0" rpy="${-pi/2} 0 ${-pi/2}"/>
+  </xacro:sensor_d435>
 </robot>

Commit message: add plugins about realsense to tb3_punptilt.gazebo

File: turtlebot3_description/urdf/turtlebot3_burger_puntilt.gazebo.xacro (robot description, xacro)
@@ -3,4 +3,6 @@
   <xacro:arg name="laser_visual" default="false"/>
   <xacro:arg name="imu_visual"   default="false"/>
+  <xacro:arg name="realsese_color_visual"   default="false"/>
+  <xacro:arg name="realsese_depth_visual"   default="true"/>
   <gazebo reference="base_link">
     <material>Gazebo/DarkGrey</material>
@@ -33,11 +35,4 @@
     <minDepth>0.001</minDepth>
     <maxVel>1.0</maxVel>
-    <material>Gazebo/FlatBlack</material>
-  </gazebo>
-  <gazebo reference="imu_link">
-    <sensor type="imu" name="imu">
-      <always_on>true</always_on>
-      <visualize>$(arg imu_visual)</visualize>
-    </sensor>
     <material>Gazebo/FlatBlack</material>
   </gazebo>
@@ -63,4 +58,11 @@
       <rosDebugLevel>na</rosDebugLevel>
     </plugin>
+  </gazebo>
+  <gazebo reference="imu_link">
+    <sensor type="imu" name="imu">
+      <always_on>true</always_on>
+      <visualize>$(arg imu_visual)</visualize>
+    </sensor>
+    <material>Gazebo/FlatBlack</material>
   </gazebo>
   <gazebo>
@@ -92,4 +94,5 @@
     </plugin>
   </gazebo>
+	<!-- LiDAR -->
   <gazebo reference="base_scan">
     <material>Gazebo/FlatBlack</material>
@@ -124,9 +127,84 @@
     </sensor>
   </gazebo>
-  <!-- <gazebo>
-    <plugin name="control" filename="libgazebo_ros_control.so"/>
-    <plugin name="joint_state_publisher" filename="libgazebo_ros_joint_state_publisher.so">
-      <jointName>base_puntilt_joint, base_realsense_joint</jointName>
-    </plugin>
-  </gazebo> -->
+	<!-- realsense -->
+	<gazebo reference="camera_color_frame">
+      <sensor type="camera" name="realsense_color">
+			<always_on>true</always_on>
+	      <visualize>$(arg realsese_color_visual)</visualize>
+        <update_rate>30.0</update_rate>
+        <camera name="realsense">
+          <pose>0 0 0 0 ${radians(-90)} ${radians(90)}</pose>
+          <horizontal_fov>1.3962634</horizontal_fov>
+          <image>
+            <width>800</width>
+            <height>600</height>
+            <format>R8G8B8</format>
+          </image>
+          <clip>
+            <near>0.02</near>
+            <far>300</far>
+          </clip>
+          <noise>
+            <type>gaussian</type>
+            <mean>0.0</mean>
+            <stddev>0.007</stddev>
+          </noise>
+        </camera>
+        <plugin name="camera_controller" filename="libgazebo_ros_camera.so">
+          <alwaysOn>true</alwaysOn>
+          <updateRate>30.0</updateRate>
+          <cameraName>		tb3_puntilt/realsense/color</cameraName>
+          <imageTopicName>	image_raw</imageTopicName>
+          <cameraInfoTopicName>camera_info</cameraInfoTopicName>
+          <frameName>camera_color_frame</frameName>
+          <hackBaseline>0.0</hackBaseline>
+          <distortionK1>0.0</distortionK1>
+          <distortionK2>0.0</distortionK2>
+          <distortionK3>0.0</distortionK3>
+          <distortionT1>0.0</distortionT1>
+          <distortionT2>0.0</distortionT2>
+        </plugin>
+      </sensor>
+    </gazebo>
+	<gazebo reference="camera_depth_frame">
+		<sensor name="depth_camera" type="depth">
+			<always_on>true</always_on>
+			<update_rate>20</update_rate>
+	      <visualize>$(arg realsese_depth_visual)</visualize>
+			<camera>
+				<horizontal_fov>1.2</horizontal_fov>
+				<image>
+				<format>R8G8B8</format>
+				<width>80</width>
+				<height>60</height>
+				</image>
+				<clip>
+				<near>0.02</near>
+				<far>300</far>
+				</clip>
+			</camera>
+			<plugin filename="libgazebo_ros_depth_camera.so" name="depth_camera_controller">
+          	<alwaysOn>true</alwaysOn>
+				<updateRate>10.0</updateRate>
+				<cameraName>tb3_puntilt/realsense/depth</cameraName>
+				<imageTopicName>color/image_raw</imageTopicName>
+				<cameraInfoTopicName>color/camera_info</cameraInfoTopicName>
+				<pointCloudTopicName>point</pointCloudTopicName>
+				<depthImageTopicName>depth/image_raw</depthImageTopicName>
+				<depthImageCameraInfoTopicName>depth/camera_info</depthImageCameraInfoTopicName>
+				<pointCloudCutoff>0.4</pointCloudCutoff>
+				<frameName>camera_depth_frame</frameName>
+				<CxPrime>0.0</CxPrime>
+				<Cx>0.0</Cx>
+				<Cy>0.0</Cy>
+				<focalLength>0.0</focalLength> <!-- use computed_focal_length -->
+				<hackBaseline>0.12</hackBaseline> <!-- use for P[3] -->
+				<distortionK1>0.05</distortionK1>
+				<distortionK2>-0.05</distortionK2>
+				<distortionK3>0.0</distortionK3>
+				<distortionT1>0.0</distortionT1>
+				<distortionT2>0.0</distortionT2>
+			</plugin>
+		</sensor>
+    </gazebo>
 </robot>

Commit message: fix realsense pulgin coordinate in tb3_burger_puntilt

File: turtlebot3_description/urdf/turtlebot3_burger_puntilt.gazebo.xacro (robot description, xacro)
@@ -134,5 +134,5 @@
         <update_rate>30.0</update_rate>
         <camera name="realsense">
-          <pose>0 0 0 0 ${radians(-90)} ${radians(90)}</pose>
+          <pose>0 0 0 0 ${radians(0)} ${radians(0)}</pose>
           <horizontal_fov>1.3962634</horizontal_fov>
           <image>
@@ -171,7 +171,9 @@
 			<always_on>true</always_on>
 			<update_rate>20</update_rate>
+			<origin xyz="0 0 0" rpy="${0} ${0} ${0}"/>
 	      <visualize>$(arg realsese_depth_visual)</visualize>
 			<camera>
 				<horizontal_fov>1.2</horizontal_fov>
+	          <pose>0 0 0 ${radians(0)} ${radians(0)} ${radians(0)}</pose>
 				<image>
 				<format>R8G8B8</format>
@@ -194,5 +196,5 @@
 				<depthImageCameraInfoTopicName>depth/camera_info</depthImageCameraInfoTopicName>
 				<pointCloudCutoff>0.4</pointCloudCutoff>
-				<frameName>camera_depth_frame</frameName>
+				<frameName>camera_depth_optical_frame</frameName>
 				<CxPrime>0.0</CxPrime>
 				<Cx>0.0</Cx>
@@ -208,3 +210,17 @@
 		</sensor>
     </gazebo>
+	<!-- launchのcontrollerとペアで使うはずだと思うんだけど，namespaceがうまく解決できなくて，うまくいかない．むしろないと動く -->
+	<!-- <gazebo>
+		<plugin name="gazebo_ros_control" filename="libgazebo_ros_control.so">
+			<robotNamespace>/burger_puntilt</robotNamespace>
+			<robotSimType>gazebo_ros_control/DefaultRobotHWSim</robotSimType>
+			<legacyModeNS>true</legacyModeNS>
+		</plugin>
+	</gazebo> -->
+	<!-- アクチュエータのない関節をpubplishするために必要らしい -->
+	<!-- <gazebo>
+      <plugin name="joint_state_publisher" filename="libgazebo_ros_joint_state_publisher.so">
+        <jointName></jointName>
+      </plugin>
+    </gazebo> -->
 </robot>

File: turtlebot3_description/urdf/turtlebot3_pizza.urdf.xacro (robot description, xacro)
@@ -50,7 +50,7 @@
       <origin xyz="0 0 0" rpy="0 0 0"/>
       <mass value="1.0"/>
-      <inertia ixx="8.7002718e-03" ixy="-4.7576583e-05" ixz="1.1160499e-04"
-               iyy="8.6195418e-03" iyz="-3.5422299e-06"
-               izz="1.4612727e-02" />
+      <inertia ixx="8.7002718e-03" ixy="-4.7576583e-05" ixz=" 1.1160499e-04"
+                                   iyy=" 8.6195418e-03" iyz="-3.5422299e-06"
+                                                        izz=" 1.4612727e-02" />
     </inertial>
   </link>
@@ -79,6 +79,6 @@
       <mass value="0.170" />
       <inertia ixx="1.1175580e-05" ixy="-4.2369783e-11" ixz="-5.9381719e-09"
-               iyy="1.1192413e-05" iyz="-1.4400107e-11"
-               izz="2.0712558e-05" />
+                                   iyy=" 1.1192413e-05" iyz="-1.4400107e-11"
+                                                        izz=" 2.0712558e-05" />
       </inertial>
   </link>
@@ -107,6 +107,6 @@
       <mass value="0.170" />
       <inertia ixx="1.1175580e-05" ixy="-4.2369783e-11" ixz="-5.9381719e-09"
-               iyy="1.1192413e-05" iyz="-1.4400107e-11"
-               izz="2.0712558e-05" />
+                                   iyy=" 1.1192413e-05" iyz="-1.4400107e-11"
+                                                        izz=" 2.0712558e-05" />
       </inertial>
   </link>
@@ -218,7 +218,7 @@
       <origin xyz="0 0 0" />
       <mass value="0.170" />
-      <inertia ixx="0.001" ixy="0.0" ixz="0.0"
-               iyy="0.001" iyz="0.0"
-               izz="0.001" />
+      <inertia ixx="0.001" ixy="0.000" ixz="0.000"
+                           iyy="0.001" iyz="0.000"
+                                       izz="0.001" />
     </inertial>
   </link>
@@ -246,7 +246,7 @@
       <origin xyz="0 0 0" />
       <mass value="0.170" />
-      <inertia ixx="0.001" ixy="0.0" ixz="0.0"
-               iyy="0.001" iyz="0.0"
-               izz="0.001" />
+      <inertia ixx="0.001" ixy="0.000" ixz="0.000"
+                           iyy="0.001" iyz="0.000"
+                                       izz="0.001" />
     </inertial>
   </link>
@@ -304,5 +304,5 @@
     <origin xyz="0.09496655 0.0 0.1375" rpy="0 0 0"/>
   </joint>
-  <xacro:sick_tim571 name="laser" ros_topic="scan"/>
+  <xacro:sick_tim551 name="laser" ros_topic="scan"/>
   <!-- z_offset: distance between base plate and laser center (= center of mesh) -->
   <!-- <link name="laser_mount_link">

Commit message: librealsense_gazebo_plugin.soを落とさないと使えないやり方

File: turtlebot3_description/urdf/turtlebot3_burger_puntilt.gazebo.xacro (robot description, xacro)
@@ -1,7 +1,7 @@
 <?xml version="1.0"?>
-<robot name="turtlebot3_burger_sim" xmlns:xacro="http://ros.org/wiki/xacro">
-  <xacro:arg name="laser_visual" default="false"/>
-  <xacro:arg name="imu_visual"   default="false"/>
-  <xacro:arg name="realsese_color_visual"   default="false"/>
+<robot name="turtlebot3_burger_puntilt" xmlns:xacro="http://ros.org/wiki/xacro">
+  <xacro:arg name="laser_visual" default="true"/>
+  <xacro:arg name="imu_visual"   default="true"/>
+  <xacro:arg name="realsese_color_visual"   default="true"/>
   <xacro:arg name="realsese_depth_visual"   default="true"/>
   <gazebo reference="base_link">
@@ -127,21 +127,38 @@
     </sensor>
   </gazebo>
+	<xacro:arg name="camera_name" default="realsense" />
+	<xacro:arg name="reference_link" default="camera_color_frame" />
+	<xacro:arg name="topics_ns" default="puntilt" />
+	<xacro:arg name="depth_optical_frame" default="camera_depth_optical_frame" />
+	<xacro:arg name="color_optical_frame" default="camera_color_optical_frame" />
+	<xacro:arg name="infrared1_optical_frame" default="camera_infra1_optical_frame" />
+	<xacro:arg name="infrared2_optical_frame" default="camera_infra2_optical_frame" />
+	<xacro:arg name="publish_pointcloud" default="true" />
 	<!-- realsense -->
-	<gazebo reference="camera_color_frame">
-      <sensor type="camera" name="realsense_color">
-			<always_on>true</always_on>
-	      <visualize>$(arg realsese_color_visual)</visualize>
-        <update_rate>30.0</update_rate>
-        <camera name="realsense">
-          <pose>0 0 0 0 ${radians(0)} ${radians(0)}</pose>
-          <horizontal_fov>1.3962634</horizontal_fov>
-          <image>
-            <width>800</width>
-            <height>600</height>
-            <format>R8G8B8</format>
-          </image>
-          <clip>
-            <near>0.02</near>
-            <far>300</far>
+   <gazebo reference="$(arg reference_link)">
+      <self_collide>0</self_collide>
+      <enable_wind>0</enable_wind>
+      <kinematic>0</kinematic>
+      <gravity>1</gravity>
+      <!--<mu>1</mu>-->
+      <mu2>1</mu2>
+      <fdir1>0 0 0</fdir1>
+      <!--<slip1>0</slip1>
+      <slip2>0</slip2>-->
+      <kp>1e+13</kp>
+      <kd>1</kd>
+      <!--<max_vel>0.01</max_vel>
+      <min_depth>0</min_depth>-->
+      <sensor name="$(arg camera_name)_color" type="camera">
+        <camera name="$(arg camera_name)">
+          <horizontal_fov>${radians(69.4)}</horizontal_fov>
+          <image>
+            <width>640</width>
+            <height>480</height>
+            <format>RGB_INT8</format>
+          </image>
+          <clip>
+            <near>0.1</near>
+            <far>100</far>
           </clip>
           <noise>
@@ -151,62 +168,99 @@
           </noise>
         </camera>
-        <plugin name="camera_controller" filename="libgazebo_ros_camera.so">
-          <alwaysOn>true</alwaysOn>
-          <updateRate>30.0</updateRate>
-          <cameraName>		tb3_puntilt/realsense/color</cameraName>
-          <imageTopicName>	image_raw</imageTopicName>
-          <cameraInfoTopicName>camera_info</cameraInfoTopicName>
-          <frameName>camera_color_frame</frameName>
-          <hackBaseline>0.0</hackBaseline>
-          <distortionK1>0.0</distortionK1>
-          <distortionK2>0.0</distortionK2>
-          <distortionK3>0.0</distortionK3>
-          <distortionT1>0.0</distortionT1>
-          <distortionT2>0.0</distortionT2>
-        </plugin>
+        <always_on>1</always_on>
+        <update_rate>30</update_rate>
+        <visualize>1</visualize>
+      </sensor>
+      <sensor name="$(arg camera_name)_ired1" type="camera">
+        <camera name="$(arg camera_name)">
+          <horizontal_fov>${radians(85.2)}</horizontal_fov>
+          <image>
+            <width>1280</width>
+            <height>720</height>
+            <format>L_INT8</format>
+          </image>
+          <clip>
+            <near>0.1</near>
+            <far>100</far>
+          </clip>
+          <noise>
+            <type>gaussian</type>
+            <mean>0.0</mean>
+            <stddev>0.05</stddev>
+          </noise>
+        </camera>
+        <always_on>1</always_on>
+        <update_rate>90</update_rate>
+        <visualize>0</visualize>
+      </sensor>
+      <sensor name="$(arg camera_name)_ired2" type="camera">
+        <camera name="$(arg camera_name)">
+          <horizontal_fov>${radians(85.2)}</horizontal_fov>
+          <image>
+            <width>1280</width>
+            <height>720</height>
+            <format>L_INT8</format>
+          </image>
+          <clip>
+            <near>0.1</near>
+            <far>100</far>
+          </clip>
+          <noise>
+            <type>gaussian</type>
+            <mean>0.0</mean>
+            <stddev>0.05</stddev>
+          </noise>
+        </camera>
+        <always_on>1</always_on>
+        <update_rate>90</update_rate>
+        <visualize>0</visualize>
+      </sensor>
+      <sensor name="$(arg camera_name)_depth" type="depth">
+        <camera name="$(arg camera_name)">
+          <horizontal_fov>${radians(85.2)}</horizontal_fov>
+          <image>
+            <width>1280</width>
+            <height>720</height>
+          </image>
+          <clip>
+            <near>0.1</near>
+            <far>100</far>
+          </clip>
+          <noise>
+            <type>gaussian</type>
+            <mean>0.0</mean>
+            <stddev>0.100</stddev>
+          </noise>
+        </camera>
+        <always_on>1</always_on>
+        <update_rate>90</update_rate>
+        <visualize>0</visualize>
       </sensor>
     </gazebo>
-	<gazebo reference="camera_depth_frame">
-		<sensor name="depth_camera" type="depth">
-			<always_on>true</always_on>
-			<update_rate>20</update_rate>
-			<origin xyz="0 0 0" rpy="${0} ${0} ${0}"/>
-	      <visualize>$(arg realsese_depth_visual)</visualize>
-			<camera>
-				<horizontal_fov>1.2</horizontal_fov>
-	          <pose>0 0 0 ${radians(0)} ${radians(0)} ${radians(0)}</pose>
-				<image>
-				<format>R8G8B8</format>
-				<width>80</width>
-				<height>60</height>
-				</image>
-				<clip>
-				<near>0.02</near>
-				<far>300</far>
-				</clip>
-			</camera>
-			<plugin filename="libgazebo_ros_depth_camera.so" name="depth_camera_controller">
-          	<alwaysOn>true</alwaysOn>
-				<updateRate>10.0</updateRate>
-				<cameraName>tb3_puntilt/realsense/depth</cameraName>
-				<imageTopicName>color/image_raw</imageTopicName>
-				<cameraInfoTopicName>color/camera_info</cameraInfoTopicName>
-				<pointCloudTopicName>point</pointCloudTopicName>
-				<depthImageTopicName>depth/image_raw</depthImageTopicName>
-				<depthImageCameraInfoTopicName>depth/camera_info</depthImageCameraInfoTopicName>
-				<pointCloudCutoff>0.4</pointCloudCutoff>
-				<frameName>camera_depth_optical_frame</frameName>
-				<CxPrime>0.0</CxPrime>
-				<Cx>0.0</Cx>
-				<Cy>0.0</Cy>
-				<focalLength>0.0</focalLength> <!-- use computed_focal_length -->
-				<hackBaseline>0.12</hackBaseline> <!-- use for P[3] -->
-				<distortionK1>0.05</distortionK1>
-				<distortionK2>-0.05</distortionK2>
-				<distortionK3>0.0</distortionK3>
-				<distortionT1>0.0</distortionT1>
-				<distortionT2>0.0</distortionT2>
-			</plugin>
-		</sensor>
+    <gazebo>
+      <plugin name="$(arg topics_ns)" filename="librealsense_gazebo_plugin.so">
+        <prefix>$(arg camera_name)</prefix>
+        <depthUpdateRate>30.0</depthUpdateRate>
+        <colorUpdateRate>30.0</colorUpdateRate>
+        <infraredUpdateRate>30.0</infraredUpdateRate>
+        <depthTopicName>depth/image_raw</depthTopicName>
+        <depthCameraInfoTopicName>depth/camera_info</depthCameraInfoTopicName>
+        <colorTopicName>color/image_raw</colorTopicName>
+        <colorCameraInfoTopicName>color/camera_info</colorCameraInfoTopicName>
+        <infrared1TopicName>infra1/image_raw</infrared1TopicName>
+        <infrared1CameraInfoTopicName>infra1/camera_info</infrared1CameraInfoTopicName>
+        <infrared2TopicName>infra2/image_raw</infrared2TopicName>
+        <infrared2CameraInfoTopicName>infra2/camera_info</infrared2CameraInfoTopicName>
+        <colorOpticalframeName>$(arg color_optical_frame)</colorOpticalframeName>
+        <depthOpticalframeName>$(arg depth_optical_frame)</depthOpticalframeName>
+        <infrared1OpticalframeName>$(arg infrared1_optical_frame)</infrared1OpticalframeName>
+        <infrared2OpticalframeName>$(arg infrared2_optical_frame)</infrared2OpticalframeName>
+        <rangeMinDepth>0.2</rangeMinDepth>
+        <rangeMaxDepth>10.0</rangeMaxDepth>
+        <pointCloud>$(arg publish_pointcloud)</pointCloud>
+        <pointCloudTopicName>depth/color/points</pointCloudTopicName>
+        <pointCloudCutoff>0.25</pointCloudCutoff>
+        <pointCloudCutoffMax>9.0</pointCloudCutoffMax>
+      </plugin>
     </gazebo>
 	<!-- launchのcontrollerとペアで使うはずだと思うんだけど，namespaceがうまく解決できなくて，うまくいかない．むしろないと動く -->
