Commit message: update params to ros2 format

File: turtlebot3_description/urdf/turtlebot3_big_wheel.gazebo.xacro (robot description, xacro)
@@ -48,7 +48,56 @@
   </gazebo>
   <gazebo reference="imu_link">
-    <sensor type="imu" name="imu">
+    <sensor name="tb3_imu" type="imu">
       <always_on>true</always_on>
       <visualize>$(arg imu_visual)</visualize>
+      <update_rate>200</update_rate>
+      <imu>
+        <angular_velocity>
+          <x>
+            <noise type="gaussian">
+              <mean>0.0</mean>
+              <stddev>2e-4</stddev>
+            </noise>
+          </x>
+          <y>
+            <noise type="gaussian">
+              <mean>0.0</mean>
+              <stddev>2e-4</stddev>
+            </noise>
+          </y>
+          <z>
+            <noise type="gaussian">
+              <mean>0.0</mean>
+              <stddev>2e-4</stddev>
+            </noise>
+          </z>
+        </angular_velocity>
+        <linear_acceleration>
+          <x>
+            <noise type="gaussian">
+              <mean>0.0</mean>
+              <stddev>1.7e-2</stddev>
+            </noise>
+          </x>
+          <y>
+            <noise type="gaussian">
+              <mean>0.0</mean>
+              <stddev>1.7e-2</stddev>
+            </noise>
+          </y>
+          <z>
+            <noise type="gaussian">
+              <mean>0.0</mean>
+              <stddev>1.7e-2</stddev>
+            </noise>
+          </z>
+        </linear_acceleration>
+      </imu>
+      <plugin name="turtlebot3_imu" filename="libgazebo_ros_imu_sensor.so">
+        <ros>
+          <!-- <namespace>/tb3</namespace> -->
+          <remapping>~/out:=imu</remapping>
+        </ros>
+      </plugin>
     </sensor>
     <material>Gazebo/Grey</material>
@@ -56,58 +105,41 @@
   <gazebo>
     <plugin name="turtlebot3_big_wheel_controller" filename="libgazebo_ros_diff_drive.so">
-      <commandTopic>cmd_vel</commandTopic>
-      <odometryTopic>odom</odometryTopic>
-      <odometryFrame>odom</odometryFrame>
-      <odometrySource>world</odometrySource>
-      <publishOdomTF>true</publishOdomTF>
-      <robotBaseFrame>base_footprint</robotBaseFrame>
-      <publishWheelTF>false</publishWheelTF>
-      <publishTf>true</publishTf>
-      <publishWheelJointState>true</publishWheelJointState>
-      <legacyMode>false</legacyMode>
-      <updateRate>30</updateRate>
-      <leftJoint>wheel_left_joint</leftJoint>
-      <rightJoint>wheel_right_joint</rightJoint>
-      <wheelSeparation>0.287</wheelSeparation>
-      <wheelDiameter>0.1245</wheelDiameter>
-      <wheelAcceleration>1</wheelAcceleration>
-      <wheelTorque>10</wheelTorque>
-      <rosDebugLevel>na</rosDebugLevel>
+      <ros>
+        <!-- <namespace>/tb3</namespace> -->
+      </ros>
+      <update_rate>30</update_rate>
+      <!-- wheels -->
+      <left_joint>wheel_left_joint</left_joint>
+      <right_joint>wheel_right_joint</right_joint>
+      <!-- kinematics -->
+      <wheel_separation>0.287</wheel_separation>
+      <wheel_diameter>0.1245</wheel_diameter>
+      <!-- limits -->
+      <max_wheel_torque>20</max_wheel_torque>
+      <max_wheel_acceleration>1.0</max_wheel_acceleration>
+      <command_topic>cmd_vel</command_topic>
+      <!-- output -->
+      <publish_odom>true</publish_odom>
+      <publish_odom_tf>true</publish_odom_tf>
+      <publish_wheel_tf>false</publish_wheel_tf>
+      <odometry_topic>odom</odometry_topic>
+      <odometry_frame>odom</odometry_frame>
+      <robot_base_frame>base_footprint</robot_base_frame>
     </plugin>
   </gazebo>
   <gazebo>
-    <plugin name="imu_plugin" filename="libgazebo_ros_imu.so">
-      <alwaysOn>true</alwaysOn>
-      <bodyName>imu_link</bodyName>
-      <frameName>imu_link</frameName>
-      <topicName>imu</topicName>
-      <serviceName>imu_service</serviceName>
-      <gaussianNoise>0.0</gaussianNoise>
-      <updateRate>0</updateRate>
-      <imu>
-        <noise>
-          <type>gaussian</type>
-          <rate>
-            <mean>0.0</mean>
-            <stddev>2e-4</stddev>
-            <bias_mean>0.0000075</bias_mean>
-            <bias_stddev>0.0000008</bias_stddev>
-          </rate>
-          <accel>
-            <mean>0.0</mean>
-            <stddev>1.7e-2</stddev>
-            <bias_mean>0.1</bias_mean>
-            <bias_stddev>0.001</bias_stddev>
-          </accel>
-        </noise>
-      </imu>
+    <plugin name="imu_plugin" filename="libgazebo_ros_imu_sensor.so">
+      <ros>
+        <!-- <namespace>/tb3</namespace> -->
+        <remapping>~/out:=imu</remapping>
+      </ros>
     </plugin>
   </gazebo>
   <xacro:if value="${lds_model=='LDS-01'}">
     <gazebo reference="base_scan">
-      <material>Gazebo/FlatBlack</material>
-      <sensor type="ray" name="lds_lfcd_sensor">
-        <pose>0 0 0 0 0 0</pose>
-        <visualize>$(arg laser_visual)</visualize>
+      <sensor name="hls_lfcd_lds" type="ray">
+        <always_on>true</always_on>
+        <visualize>true</visualize>
+        <pose>-0.064 0 0.121 0 0 0</pose>
         <update_rate>5</update_rate>
         <ray>
@@ -115,6 +147,6 @@
             <horizontal>
               <samples>360</samples>
-              <resolution>1</resolution>
-              <min_angle>0.0</min_angle>
+              <resolution>1.000000</resolution>
+              <min_angle>0.000000</min_angle>
               <max_angle>6.28319</max_angle>
             </horizontal>
@@ -123,5 +155,5 @@
             <min>0.150</min>
             <max>3.5</max>
-            <resolution>0.015</resolution>
+            <resolution>0.015000</resolution>
           </range>
           <noise>
@@ -131,17 +163,22 @@
           </noise>
         </ray>
-        <plugin name="gazebo_ros_lds_lfcd_controller" filename="libgazebo_ros_laser.so">
-          <topicName>scan</topicName>
-          <frameName>base_scan</frameName>
+        <plugin name="turtlebot3_laserscan" filename="libgazebo_ros_ray_sensor.so">
+          <ros>
+            <!-- <namespace>/tb3</namespace> -->
+            <remapping>~/out:=scan</remapping>
+          </ros>
+          <output_type>sensor_msgs/LaserScan</output_type>
+          <frame_name>base_scan</frame_name>
         </plugin>
       </sensor>
+      <material>Gazebo/FlatBlack</material>
     </gazebo>
   </xacro:if>
   <xacro:if value="${lds_model=='LDS-02'}">
     <gazebo reference="base_scan">
-      <material>Gazebo/FlatBlack</material>
-      <sensor type="ray" name="lds_lfcd_sensor">
-        <pose>0 0 0 0 0 0</pose>
-        <visualize>$(arg laser_visual)</visualize>
+      <sensor name="hls_lfcd_lds" type="ray">
+        <always_on>true</always_on>
+        <visualize>true</visualize>
+        <pose>-0.064 0 0.121 0 0 0</pose>
         <update_rate>5</update_rate>
         <ray>
@@ -149,6 +186,6 @@
             <horizontal>
               <samples>360</samples>
-              <resolution>1</resolution>
-              <min_angle>0.0</min_angle>
+              <resolution>1.000000</resolution>
+              <min_angle>0.000000</min_angle>
               <max_angle>6.28319</max_angle>
             </horizontal>
@@ -157,5 +194,5 @@
             <min>0.20</min>
             <max>8.0</max>
-            <resolution>0.015</resolution>
+            <resolution>0.015000</resolution>
           </range>
           <noise>
@@ -165,9 +202,14 @@
           </noise>
         </ray>
-        <plugin name="gazebo_ros_lds_lfcd_controller" filename="libgazebo_ros_laser.so">
-          <topicName>scan</topicName>
-          <frameName>base_scan</frameName>
+        <plugin name="turtlebot3_laserscan" filename="libgazebo_ros_ray_sensor.so">
+          <ros>
+            <!-- <namespace>/tb3</namespace> -->
+            <remapping>~/out:=scan</remapping>
+          </ros>
+          <output_type>sensor_msgs/LaserScan</output_type>
+          <frame_name>base_scan</frame_name>
         </plugin>
       </sensor>
+      <material>Gazebo/FlatBlack</material>
     </gazebo>
   </xacro:if>

Commit message: Modified colors

File: turtlebot3_description/urdf/turtlebot3_big_wheel.gazebo.xacro (robot description, xacro)
@@ -172,4 +172,22 @@
     </gazebo>
   </xacro:if>
+  <gazebo reference="rpi_link">
+    <mu1>0.1</mu1>
+    <mu2>0.1</mu2>
+    <kp>1000000.0</kp>
+    <kd>100.0</kd>
+    <minDepth>0.001</minDepth>
+    <maxVel>1.0</maxVel>
+    <material>Gazebo/DarkGrey</material>
+  </gazebo>
+  <gazebo reference="battery_link">
+    <mu1>0.1</mu1>
+    <mu2>0.1</mu2>
+    <kp>1000000.0</kp>
+    <kd>100.0</kd>
+    <minDepth>0.001</minDepth>
+    <maxVel>1.0</maxVel>
+    <material>Gazebo/DarkGrey</material>
+  </gazebo>
   <gazebo reference="base_camera_link">
     <material>Gazebo/DarkGrey</material>

File: turtlebot3_description/urdf/turtlebot3_big_wheel.urdf.xacro (robot description, xacro)
@@ -210,4 +210,5 @@
         <box size="0.055 0.040 0.02"/>
       </geometry>
+      <material name="dark"/>
     </visual>
     <inertial>
@@ -230,4 +231,5 @@
         <box size="0.08 0.03 0.02"/>
       </geometry>
+      <material name="dark"/>
     </visual>
     <inertial>

File: turtlebot3_description/urdf/turtlebot3_big_wheel_3rs.urdf.xacro (robot description, xacro)
@@ -290,4 +290,5 @@
         <box size="0.055 0.040 0.02"/>
       </geometry>
+      <material name="dark"/>
     </visual>
     <inertial>
@@ -310,4 +311,5 @@
         <box size="0.08 0.03 0.02"/>
       </geometry>
+      <material name="dark"/>
     </visual>
     <inertial>

File: turtlebot3_description/urdf/turtlebot3_big_wheel_for_open_manipulator.urdf.xacro (robot description, xacro)
@@ -201,4 +201,46 @@
     </collision> -->
   </link>
+  <joint name="rpi_joint" type="fixed">
+    <parent link="base_link"/>
+    <child link="rpi_link"/>
+    <origin xyz="-0.13 0.0 0.05" rpy="0 0 0"/>
+  </joint>
+  <link name="rpi_link">
+    <visual>
+      <origin xyz="0 0.00175 0" rpy="0 0 0"/>
+      <geometry>
+        <box size="0.055 0.040 0.02"/>
+      </geometry>
+      <material name="dark"/>
+    </visual>
+    <inertial>
+      <origin xyz="0 0 0"/>
+      <mass value="0.047"/>
+      <inertia ixx="0.001" ixy="0.0" ixz="0.0"
+               iyy="0.001" iyz="0.0"
+               izz="0.001" />
+    </inertial>
+  </link>
+  <joint name="battery_joint" type="fixed">
+    <parent link="base_link"/>
+    <child link="battery_link"/>
+    <origin xyz="-0.13 0.0 0.02" rpy="0 0 0"/>
+  </joint>
+  <link name="battery_link">
+    <visual>
+      <origin xyz="0 0.00175 0" rpy="0 0 0"/>
+      <geometry>
+        <box size="0.08 0.03 0.02"/>
+      </geometry>
+      <material name="dark"/>
+    </visual>
+    <inertial>
+      <origin xyz="0 0 0" />
+      <mass value="0.10" />
+      <inertia ixx="0.001" ixy="0.0" ixz="0.0"
+               iyy="0.001" iyz="0.0"
+               izz="0.001" />
+    </inertial>
+  </link>
   <xacro:sensor_d435 parent="base_camera_link" use_nominal_extrinsics="$(arg use_nominal_extrinsics)" add_plug="$(arg add_plug)" use_mesh="$(arg use_mesh)">
     <origin xyz="0.016 0.03 0.0" rpy="0 0 0"/>
