Commit message: small fix

File: turtlebot3_description/urdf/dynamixel/_2XL430.urdf.xacro (robot description, xacro)
@@ -43,4 +43,7 @@
 					<mesh filename="package://turtlebot3_description/${path_to_stl}" />
 				</geometry>
+				<material name="gray">
+					<color rgba="0.8 0.8 0.8 0.5"/>
+				</material>
 			</visual>
 			<collision>
@@ -51,5 +54,4 @@
 				</geometry>
 			</collision>
-			<material name="gray"/>
 		</link>
 		<!--あとでgazebo.xacroに入れる-->

File: turtlebot3_description/urdf/dynamixel/dynamixel_2XL430_sample_macro.urdf.xacro (robot description, xacro)
@@ -19,6 +19,12 @@
 				<cylinder length="0.001" radius="0.01"/>
 			</geometry>
-			<material name="orange"/>
+			<material name="red"/>
 		</visual>
 	</link>
+	<gazebo reference="base">
+		<material>Gazebo/Orange</material>
+	</gazebo>
+	<gazebo reference="hone">
+		<material>Gazebo/Red</material>
+	</gazebo>
 </robot>

File: turtlebot3_description/urdf/turtlebot3_burger_puntilt.urdf.xacro (robot description, xacro)
@@ -3,6 +3,6 @@
   <xacro:include filename="$(find turtlebot3_description)/urdf/common_properties.xacro"/>
   <xacro:include filename="$(find turtlebot3_description)/urdf/turtlebot3_burger_puntilt.gazebo.xacro"/>
+	<xacro:include filename="$(find turtlebot3_description)/urdf/dynamixel/_2XL430.urdf.xacro"/>
   <xacro:include filename="$(find realsense2_description)/urdf/_d435.urdf.xacro" />
-	<xacro:include filename="$(find turtlebot3_description)/urdf/_2XL430.urdf.xacro"/>
   <!-- realsense 関連の引数 -->
   <xacro:arg name="use_nominal_extrinsics" default="true"/>
